File: electronics/Base/view_base.kicad_pcb (KiCad board)
At the start: 4 copper layers, 81.2 x 81.2 mm, 55 parts, among them J1 BLDC, J2 USB_C_Receptacle_USB2.0, J3 Conn_01x04_Male, J5 Conn_01x04_Male, J6 Conn_01x07_Male, J7 Conn_01x12_Male, U1 MT6701-CT, U2 STM32F411CEU6, U3 CH340C, U4 BMI088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

Commit message: add stuff
Routing:
- net /USB_D-: track 15.1 -> 15.7 mm
Changed lines of the file:
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@@
       (drillshape 0)
       (scaleselection 1)
-      (outputdirectory "gerber/")
+      (outputdirectory "../jlc/base/")
     )
   )
@@
     (fp_line (start -4.999999 33.9) (end 4.999999 33.9) (layer "B.Fab") (width 0.2))
     (fp_arc (start 13.514575 -8.564826) (mid 14.706493 -6.302305) (end 15.522725 -3.878787) (layer "B.Fab") (width 0.2))
-    (fp_arc (start 15.522725 3.878788) (mid 14.706493 6.302306) (end 13.514574 8.564827) (layer "B.Fab") (width 0.2))
+    (fp_arc (start 15.522725 3.878788) (mid 14.706494 6.302306) (end 13.514574 8.564827) (layer "B.Fab") (width 0.2))
     (fp_arc (start -16.770509 -4.999999) (mid -15.856214 -7.404757) (end -14.599229 -9.649481) (layer "B.Fab") (width 0.2))
     (fp_arc (start -4.999999 16.770509) (mid -7.404757 15.856214) (end -9.649481 14.599229) (layer "B.Fab") (width 0.2))
@@
     (fp_arc (start -3.5 -16.007811) (mid -3.605914 -15.700082) (end -3.878787 -15.522725) (layer "B.Fab") (width 0.2))
     (fp_arc (start 4.999999 -16.770509) (mid 7.404757 -15.856214) (end 9.649481 -14.599229) (layer "B.Fab") (width 0.2))
-    (fp_arc (start 3.878788 -15.522725) (mid 6.302306 -14.706493) (end 8.564827 -13.514574) (layer "B.Fab") (width 0.2))
+    (fp_arc (start 3.878788 -15.522725) (mid 6.302306 -14.706494) (end 8.564827 -13.514574) (layer "B.Fab") (width 0.2))
     (fp_arc (start 9.649481 14.599229) (mid 7.404757 15.856214) (end 4.999999 16.770509) (layer "B.Fab") (width 0.2))
     (fp_arc (start -13.514575 8.564826) (mid -14.706493 6.302305) (end -15.522725 3.878787) (layer "B.Fab") (width 0.2))
@@
   (segment (start 95.325 133) (end 96.25 132.075) (width 0.15) (layer "F.Cu") (net 2))
   (segment (start 98.75 133.255) (end 98.75 133.85) (width 0.15) (layer "F.Cu") (net 2))
-  (segment (start 99.25 132.25) (end 99.5 132) (width 0.15) (layer "F.Cu") (net 3))
+  (segment (start 100.25 133.85) (end 100.25 132.25) (width 0.15) (layer "F.Cu") (net 3))
+  (segment (start 98.35 132.35) (end 97.595 131.595) (width 0.15) (layer "F.Cu") (net 3))
+  (segment (start 100.25 132.25) (end 100 132) (width 0.15) (layer "F.Cu") (net 3))
   (segment (start 96.195 131.295) (end 96.195 131.067737) (width 0.15) (layer "F.Cu") (net 3))
-  (segment (start 100 132) (end 100.25 132.25) (width 0.15) (layer "F.Cu") (net 3))
+  (segment (start 98.495 131.595) (end 97.595 131.595) (width 0.15) (layer "F.Cu") (net 3))
+  (segment (start 100 132) (end 98.9 132) (width 0.15) (layer "F.Cu") (net 3))
   (segment (start 95.295 131.595) (end 94.485788 131.595) (width 0.15) (layer "F.Cu") (net 3))
-  (segment (start 100.25 132.25) (end 100.25 133.85) (width 0.15) (layer "F.Cu") (net 3))
-  (segment (start 99.25 133.85) (end 99.25 132.25) (width 0.15) (layer "F.Cu") (net 3))
-  (segment (start 99.5 132) (end 100 132) (width 0.15) (layer "F.Cu") (net 3))
+  (segment (start 99.25 133.25) (end 98.35 132.35) (width 0.15) (layer "F.Cu") (net 3))
+  (segment (start 98.9 132) (end 98.495 131.595) (width 0.15) (layer "F.Cu") (net 3))
   (segment (start 97.595 131.595) (end 96.495 131.595) (width 0.15) (layer "F.Cu") (net 3))
   (segment (start 99.25 133.85) (end 99.25 133.25) (width 0.15) (layer "F.Cu") (net 3))
+  (segment (start 99.25 133.85) (end 99.25 133.330489) (width 0.15) (layer "F.Cu") (net 3))
   (segment (start 95.595 131.067737) (end 95.595 131.295) (width 0.15) (layer "F.Cu") (net 3))
-  (segment (start 99.25 133.25) (end 97.595 131.595) (width 0.15) (layer "F.Cu") (net 3))
   (segment (start 94.485788 131.595) (end 90.975 131.595) (width 0.15) (layer "F.Cu") (net 3))
   (arc (start 96.195 131.067737) (mid 96.107132 130.855605) (end 95.895 130.767737) (width 0.15) (layer "F.Cu") (net 3))
