File: electronics/LiDAR/lidar.kicad_pcb (KiCad board)
At the start: 4 copper layers, 18 x 26 mm, 38 parts, among them J1 Conn_01x12_Male, U1 OPT3101RHFR

Commit message: add stuff
Routing:
- net GND: track 47.2 -> 46.4 mm
Changed lines of the file:
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@@
     (pad_to_mask_clearance 0)
     (pcbplotparams
-      (layerselection 0x000fcff_ffffffff)
+      (layerselection 0x7fcffff_ffffffff)
       (disableapertmacros false)
       (usegerberextensions false)
@@
       (drillshape 0)
       (scaleselection 1)
-      (outputdirectory "gerber/")
+      (outputdirectory "../jlc/lidar/")
     )
   )
@@
     (pad "2" smd rect locked (at 0.455 0 270) (size 0.49 0.6) (layers "F.Cu" "F.Paste" "F.Mask")
       (net 9 "/VDD_EXT_3P3") (pintype "passive") (solder_mask_margin 0.102))
+    (model "D:/Pasteurized/FIBO Edu/Sem 3.1/EmbeddedSys/ROBKNOBv01/Kicad/BEADC1005X50N/NFZ15SR262SN10D.STEP"
+      (offset (xyz 0 -0.275 0.2))
+      (scale (xyz 1 1 1))
+      (rotate (xyz 0 0 0))
+    )
   )
   (footprint "BEADC1005X50N:BEADC1005X50N" (layer "F.Cu")
@@
       (rotate (xyz 0 0 0))
     )
+    (model "D:/Pasteurized/FIBO Edu/Sem 3.1/EmbeddedSys/ROBKNOBv01/Kicad/OPT3101RHFR/CC2520RHDRG4.STEP"
+      (offset (xyz 0 0 0))
+      (scale (xyz 1 1 1))
+      (rotate (xyz -90 0 0))
+    )
   )
   (footprint "Capacitor_SMD:C_0402_1005Metric" (layer "F.Cu")
@@
       (rotate (xyz 0 0 0))
     )
-    (model "D:/Pasteurized/FIBO Edu/Sem 3.1/EmbeddedSys/Kicad/fpcconncad/52207-1260.stp"
+    (model "D:/Pasteurized/FIBO Edu/Sem 3.1/EmbeddedSys/ROBKNOBv01/Kicad/fpcconncad/52207-1260.stp"
       (offset (xyz 0 -3.5 1.3))
       (scale (xyz 1 1 1))
@@
   (via (at 140.2 75.6) (size 0.8) (drill 0.4) (layers "F.Cu" "B.Cu") (net 5))
   (via (at 129.4 90.4) (size 0.4) (drill 0.3) (layers "F.Cu" "B.Cu") (free) (net 5))
-  (via (at 131.7 84.3) (size 0.4) (drill 0.3) (layers "F.Cu" "B.Cu") (free) (net 5))
+  (via (at 129.5 84.4) (size 0.4) (drill 0.3) (layers "F.Cu" "B.Cu") (free) (net 5))
   (via (at 141 77.5) (size 0.8) (drill 0.4) (layers "F.Cu" "B.Cu") (net 5))
   (via (at 129.4 85.7) (size 0.4) (drill 0.3) (layers "F.Cu" "B.Cu") (free) (net 5))
   (via (at 139.8 89) (size 0.4) (drill 0.3) (layers "F.Cu" "B.Cu") (free) (net 5))
   (via (at 132.6 85.7) (size 0.4) (drill 0.3) (layers "F.Cu" "B.Cu") (free) (net 5))
-  (segment (start 139.5 74.9) (end 132.4 74.9) (width 0.25) (layer "B.Cu") (net 5))
-  (segment (start 140.2 75.6) (end 139.5 74.9) (width 0.25) (layer "B.Cu") (net 5))
-  (segment (start 129.1 81.7) (end 131.7 84.3) (width 0.25) (layer "B.Cu") (net 5))
-  (segment (start 132.4 74.9) (end 129.1 78.2) (width 0.25) (layer "B.Cu") (net 5))
+  (segment (start 129.5 84.4) (end 129.5 82.1) (width 0.25) (layer "B.Cu") (net 5))
+  (segment (start 129.1 78.2) (end 132.4 74.9) (width 0.25) (layer "B.Cu") (net 5))
+  (segment (start 129.5 82.1) (end 129.1 81.7) (width 0.25) (layer "B.Cu") (net 5))
+  (segment (start 139.5 74.9) (end 140.2 75.6) (width 0.25) (layer "B.Cu") (net 5))
+  (segment (start 129.1 81.7) (end 129.1 78.2) (width 0.25) (layer "B.Cu") (net 5))
   (segment (start 141 77.3) (end 141 77.5) (width 0.25) (layer "B.Cu") (net 5))
   (segment (start 139.8 89) (end 137.9 90.9) (width 0.25) (layer "B.Cu") (net 5))
   (segment (start 140.2 75.6) (end 141 76.4) (width 0.25) (layer "B.Cu") (net 5))
   (segment (start 137.9 90.9) (end 130.6 90.9) (width 0.25) (layer "B.Cu") (net 5))
+  (segment (start 132.4 74.9) (end 139.5 74.9) (width 0.25) (layer "B.Cu") (net 5))
   (segment (start 141 76.4) (end 141 77.3) (width 0.25) (layer "B.Cu") (net 5))
-  (segment (start 129.1 78.2) (end 129.1 81.7) (width 0.25) (layer "B.Cu") (net 5))
   (segment (start 132.8393 86.8612) (end 132.396 87.3047) (width 0.25) (layer "F.Cu") (net 6))
   (segment (start 131.52 91.62) (end 131.8 91.9) (width 0.25) (layer "F.Cu") (net 6))
